File: rp2040-led-board-schematics-v02.kicad_sch (KiCad schematic)
At the start: 98 parts, among them IC1 UA78L05CDR, J1 GPIO, J10 LED1Terminal, J2 PWR_IN, J3 LED1Terminal, J4 LED1Terminal, J5 LED1Terminal, J6 LED1Terminal, J7 LED1Terminal, J8 LED1Terminal, J9 LED1Terminal, SW1 Button, SW2 PEC16-2115F-S0012, U1 Pico, U2 MAX485E, U3 MAX485E, U4 MAX485E, U5 MAX485E, U6 ENC28J60, U7 MAX485E, U8 MAX485E

Commit message: footprints ok
Parts:
- removed IC1: UA78L05CDR, SamacSys_Parts:SOIC127P600X175-8N, symbol Frangitron:UA78L05CDR
- removed R25: 1k, Resistor_SMD:R_0805_2012Metric, symbol Device:R_Small
- removed R25: 10k, Resistor_SMD:R_0805_2012Metric, symbol Device:R_Small
- removed R36: 120, Resistor_SMD:R_0805_2012Metric, symbol Device:R_Small
- removed SW1: Button, Button_Switch_THT:SW_Tactile_SKHH_Angled, symbol Switch:SW_Push
- removed SW2: PEC16-2115F-S0012, SamacSys_Parts:PEC162115FS0012, symbol SamacSys_Parts:PEC16-2115F-S0012
- added C14: 220nF, Capacitor_SMD:C_0603_1608Metric, symbol Device:C_Small
- added C15, C2: 100nF, Capacitor_SMD:C_0603_1608Metric, symbol Device:C_Small
- added C3: 10uF, Capacitor_SMD:C_0402_1005Metric, symbol Device:C_Small
- added H1 (x2): ~, Frangitron:frangitron_logo_16mm, symbol Frangitron:Frangitron_logo
- added J11: MainBoard, Connector_PinHeader_2.54mm:PinHeader_2x05_P2.54mm_Vertical, symbol Connector_Generic:Conn_02x05_Odd_Even
- added J12: FrontPanel, Connector_PinHeader_2.54mm:PinHeader_2x05_P2.54mm_Vertical, symbol Connector_Generic:Conn_02x05_Odd_Even
- added J14: ReceiverData, Frangitron:ScrewTerminal_01x02_5.08_Amphenol, symbol Connector:Screw_Terminal_01x02
- added J15: ReceiverRS485, Frangitron:ScrewTerminal_01x03_5.08_Amphenol, symbol Connector:Screw_Terminal_01x03
- added JP3: 1-2 12V, Jumper:SolderJumper-3_P2.0mm_Open_TrianglePad1.0x1.5mm_NumberLabels, symbol Jumper:SolderJumper_3_Open
- added JP4: 12V, Jumper:SolderJumper-2_P1.3mm_Open_Pad1.0x1.5mm, symbol Jumper:SolderJumper_2_Open
- added R10, R9: 20K, Resistor_SMD:R_0402_1005Metric, symbol Device:R_Small
- added R25: 1k, Resistor_SMD:R_0402_1005Metric, symbol Device:R_Small
- added R25: 10k, Resistor_SMD:R_0402_1005Metric, symbol Device:R_Small
- added R6 (x2), R8: 10K, Resistor_SMD:R_0402_1005Metric, symbol Device:R_Small
- added R7: 120, Resistor_SMD:R_0402_1005Metric, symbol Device:R_Small
- added SW1: Button, Frangitron:C&K_PushButtonSwitch_SPST_D6C90F2LFS, symbol Switch:SW_MEC_5E
- added SW2: PEC16, SamacSys_Parts:PEC164120FS0012, symbol SamacSys_Parts:PEC16-4220F-S0024
- added U11, U14: LM7805, Package_TO_SOT_SMD:TO-252-2, symbol Regulator_Linear:LM7805_TO220
- added U4: MAX485E, Package_SO:SOIC-8_3.9x4.9mm_P1.27mm, symbol Interface_UART:MAX485E
- C10, C12, C2, C4, C6, C8, C9: footprint Capacitor_SMD:C_0402_1005Metric -> Capacitor_SMD:C_0603_1608Metric
- C14: value 100nF -> 220nF; footprint Capacitor_SMD:C_0402_1005Metric -> Capacitor_SMD:C_0603_1608Metric
- C15: value 10uF -> 100nF; footprint Capacitor_SMD:C_0402_1005Metric -> Capacitor_SMD:C_0603_1608Metric
- DS1: footprint SamacSys_Parts:NHD0216AWIB3 -> Frangitron:NewHaven-OLED-NHD-0216AW-IB3; URL (none) -> https://www.mouser.fr/ProductDetail/Newhaven-Display/NHD-02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
- J10, J3, J4, J5, J6, J7, J8, J9: footprint SHDR3W110P0X508_1X3_1524X810X1015P -> Frangitron:ScrewTerminal_01x03_5.08_Amphenol; URL (none) -> https://www.mouser.fr/ProductDetail/Amphenol-Anytek/VI03215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
- J2: footprint 5442206 -> Frangitron:ScrewTerminal_01x02_5.08_Amphenol; URL (none) -> https://www.mouser.fr/ProductDetail/Amphenol-Anytek/VI02215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
- R10, R13, R14, R15, R18, R19, R20, R23, R24, R25, R28, R29, R30, R33, R34, R35, R7, R9: footprint Resistor_SMD:R_0805_2012Metric -> Resistor_SMD:R_0402_1005Metric
- R11, R12, R16, R17, R21, R22, R26, R27, R31, R32, R6, R8: footprint Resistor_SMD:R_0603_1608Metric -> Resistor_SMD:R_0402_1005Metric
- U2, U3, U4, U5, U7, U8: footprint SamacSys_Parts:SOIC127P600X175-8N -> Package_SO:SOIC-8_3.9x4.9mm_P1.27mm
Connections:
- net +12V: now also U11.1 (VI)
- net +3V3: now also J11.1 (Pin_1), J12.1 (Pin_1), R25.1
- net GND: now also J11.10 (Pin_10), J12.10 (Pin_10), SW1.2, SW2.C1, SW2.E1, U11.2 (GND)
- net at R25.2: now also SW2.B1
- net at R25.2: now also SW2.A1
- net at C15.1, JP2.1 (A): now also U11.3 (VO)
- net at R25.2: now also SW1.3 (K)
- net EncoderA renamed FPEncoderA
- net FPEncoderA: now also J11.6 (Pin_6); no longer U1.1 (GPIO0)
- net EncoderB renamed FPEncoderB
- net FPEncoderB: now also J11.7 (Pin_7); no longer U1.2 (GPIO1)
- net EncoderS renamed FPEncoderS
- net FPEncoderS: now also J11.5 (Pin_5), R25.2, R25.2; no longer U1.4 (GPIO2)
- net PI i2c0 RST renamed FPDisplayRST
- net FPDisplayRST: now also J11.2 (Pin_2); no longer U1.5 (GPIO3)
- net PI i2c0 SCL renamed FPDisplaySDA
- net FPDisplaySDA: now also J11.3 (Pin_3); no longer U1.7 (GPIO5)
- net PI i2c0 SDA renamed FPDisplaySCL
- net FPDisplaySCL: now also J11.4 (Pin_4); no longer U1.6 (GPIO4)
- net SwitchPush renamed FPSwitchPush
- net FPSwitchPush: now also J11.8 (Pin_8); no longer U1.19 (GPIO14)
- new net: C15.1, JP4.2 (B), U14.3 (VO)
- new net: R8.2, U4.4 (DI)
- new net: J14.2 (Pin_2), R6.2, U4.1 (RO)
- new net: J15.3 (Pin_3), R7.2, R9.2, U4.6 (A)
- new net: J15.2 (Pin_2), R10.1, R7.1, U4.7 (B)
- new net: J15.1 (Pin_1), JP3.2 (C)
- new net: R25.1, SW2.D1
- new net: C14.1, JP3.1 (A), U14.1 (VI)
- new net MBDisplayRST: J12.2 (Pin_2), U1.5 (GPIO3)
- new net MBDisplaySCL: J12.4 (Pin_4), U1.7 (GPIO5)
- new net MBDisplaySDA: J12.3 (Pin_3), U1.6 (GPIO4)
- new net MBEncoderA: J12.6 (Pin_6), U1.1 (GPIO0)
- new net MBEncoderB: J12.7 (Pin_7), U1.2 (GPIO1)
- new net MBEncoderS: J12.5 (Pin_5), U1.4 (GPIO2)
- new net MBSwitchPush: J12.8 (Pin_8), U1.19 (GPIO14)
- new net Recv5 +5V: C2.1, C3.1, JP3.3 (B), JP4.1 (A), R6.1, R6.1, R8.1, R9.1, U4.8 (VCC)
- new net Recv5 GND: C14.2, C15.2, C2.2, C3.2, J14.1 (Pin_1), R10.2, R6.2, U14.2 (GND), U4.2 (~{RE}), U4.3 (DE), U4.5 (GND)
- no-connect marks 14 -> 16
Other:
- note added: "Connector to Front Panel"
- note added: "Connector to Main Board"
- note added: "Front Panel"
- note added: "LED 1 transmitter (RS485)"
- note added: "LED 2 transmitter (RS485)"
- note added: "LED 3 transmitter (RS485)"
- note added: "LED 4 transmitter (RS485)"
- note added: "LED 5 transmitter (RS485)"
- note added: "LED 6 transmitter (RS485)"
- note added: "LED 7 transmitter (RS485)"
- note added: "LED 8 transmitter (RS485)"
- note added: "LED Receivers 5V/12V"
- note added: "Main Board"
- note added: "Misc"
- note added: "current draw: ~100mA 3V3 rail max draw: 300mA"
- note added: "current draw: ~5.5mA"
- note added: "current output: ~1A"
- note added: "total current draw: ~400mA"
- note removed: "LED 1 RS485 output"
- note removed: "LED 2 RS485 output"
- note removed: "LED 3 RS485 output"
- note removed: "LED 4 RS485 output"
- note removed: "LED 5 RS485 output"
- note removed: "LED 6 RS485 output"
- note removed: "LED 7 RS485 output"
- note removed: "LED 8 RS485 output"
- note removed: "LED Connectors"
- note removed: "Notes & Stuff"
- note removed: "current draw: ~100mA"
- note removed: "current output: 100 mA 3V3 rail max draw: 300mA"
- note removed: "total current draw: ~350mA"
- moved on the sheet: C10, C11, C12, C13, C14, C15, C2, C3, C4, C5, C6, C7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

Commit message: main board PCB done (needs checking)
Parts:
- removed C10, C12 (x2), C2, C4, C6 (x2), C8, C9 (x4): 100nF, Capacitor_SMD:C_0603_1608Metric, symbol Device:C_Small
- removed C13 (x2), C3, C5, C7 (x2), C9: 10uF, Capacitor_SMD:C_0402_1005Metric, symbol Device:C_Small
- removed J1: GPIO, Connector_PinHeader_2.54mm:PinHeader_2x07_P2.54mm_Vertical, symbol Connector_Generic:Conn_02x07_Odd_Even
- removed J10, J3, J4, J5, J6, J7, J8, J9: LED1Terminal, Frangitron:ScrewTerminal_01x03_5.08_Amphenol, symbol Connector:Screw_Terminal_01x03
- removed R10, R13, R14, R18 (x2), R19 (x2), R28, R29, R33 (x2), R34 (x2), R9: 20K, Resistor_SMD:R_0402_1005Metric, symbol Device:R_Small
- removed R11, R12, R16 (x2), R17 (x2), R26, R27, R31 (x2), R32 (x2), R6, R8: 10K, Resistor_SMD:R_0402_1005Metric, symbol Device:R_Small
- removed R15, R20 (x2), R25, R30, R35 (x2), R7: 120, Resistor_SMD:R_0402_1005Metric, symbol Device:R_Small
- removed R25 (x4): 1k, Resistor_SMD:R_0402_1005Metric, symbol Device:R_Small
- removed R25 (x4): 10k, Resistor_SMD:R_0402_1005Metric, symbol Device:R_Small
- removed U2, U3 (x2), U4, U5, U7, U8 (x2): MAX485E, Package_SO:SOIC-8_3.9x4.9mm_P1.27mm, symbol Interface_UART:MAX485E
- added C12, C13, C22: 100nF, Capacitor_SMD:C_0603_1608Metric, symbol Device:C_Small
- added FM1, FM2, FM3: Fiducial, Fiducial:Fiducial_1mm_Mask2mm, symbol Mechanical:Fiducial
- added H1, H2, H4, H5: MountingHole_Pad, MountingHole:MountingHole_3.2mm_M3_Pad, symbol Mechanical:MountingHole_Pad
- added R1, R25: 10k, Resistor_SMD:R_0402_1005Metric, symbol Device:R_Small
- added R19, R20: 1k, Resistor_SMD:R_0402_1005Metric, symbol Device:R_Small
- C11: value 10uF -> 100nF; footprint Capacitor_SMD:C_0402_1005Metric -> Capacitor_SMD:C_0603_1608Metric
- DS1: footprint Frangitron:NewHaven-OLED-NHD-0216AW-IB3 -> NHD0216AWIB3
- R21, R22: value 10K -> 1k; LCSC Part # C15401 -> C4328; LCSC Part Number C15401 -> C4328
- R23, R24: value 20K -> 10k
- SW2: footprint SamacSys_Parts:PEC164120FS0012 -> PEC164120FS0012
- U1: footprint MCU_RaspberryPi_and_Boards:RPi_Pico_SMD_TH -> RPi_Pico:RPi_Pico_SMD_TH
- U1: renamed from U11; footprint Package_TO_SOT_SMD:TO-252-2 -> Package_TO_SOT_SMD:SOT-223
- U13: renamed from U14; footprint Package_TO_SOT_SMD:TO-252-2 -> Package_TO_SOT_SMD:SOT-223
- renumbered J2 to J1, J15 to J12, J11 to J13, J12 to J5, J14 to J8, JP2 to JP1, JP1 to JP2
Connections:
- net +3.3VADC: no longer U1.35 (ADC_VREF)
- net +3V3: now also R23.1, R24.1, R1.1, R25.1; no longer DS1.2 (VDD_SEL), DS1.3 (VDDIO), J13.1 (Pin_1)
- net +5V: no longer C11.1, R21.1, R22.1, R23.1
- net FPEncoderA: now also SW2.A1
- net FPEncoderB: now also SW2.B1
- net FPEncoderS: now also SW2.D1
- net FPSwitchPush: now also SW1.3 (K)
- net GND: now also C12.2, C13.2, C22.2, H1.1, H2.1, H4.1, H5.1; no longer DS1.1 (GND), DS1.4 (SA0), J13.10 (Pin_10), R24.2, SW1.2, SW2.C1, SW2.E1
- net GNDA: no longer U1.33 (AGND)
- net LED4 out: no longer R22.2
- net MBEncoderA: now also R21.2; no longer U1.1 (GPIO0)
- net MBEncoderB: now also R22.2; no longer U1.2 (GPIO1)
- net MBEncoderS: now also R19.1; no longer U1.4 (GPIO2)
- net MBSwitchPush: now also R20.2; no longer U1.19 (GPIO14)
- net MCUSwitchPush: now reaches R23.2
- net MCUSwitchPush: now also U1.19 (GPIO14), C22.1, R20.1
- net GP15: no longer names the net of U1.20 (GPIO15)
- net GP20: no longer names the net of U1.26 (GPIO20)
- net GP21: no longer names the net of U1.27 (GPIO21)
- net GP22: no longer names the net of U1.29 (GPIO22)
- net GP26_ADC0: no longer names the net of U1.31 (GPIO26_ADC0)
- net GP27_ADC1: no longer names the net of U1.32 (GPIO27_ADC1)
- net GP28_ADC2: no longer names the net of U1.34 (GPIO28_ADC2)
- net MBDisplayRST renamed MCUDisplayRST
- net MBDisplaySCL renamed MCUDisplaySCL
- net MBDisplaySDA renamed MCUDisplaySDA
- new net FP +3V3: DS1.2 (VDD_SEL), DS1.3 (VDDIO), J13.1 (Pin_1)
- new net FP GND: DS1.1 (GND), DS1.4 (SA0), J13.10 (Pin_10), SW1.2, SW2.C1, SW2.E1
- new net MCUEncoderA: C12.1, R21.1, R24.2, U1.1 (GPIO0)
- new net MCUEncoderB: C13.1, R22.1, R25.2, U1.2 (GPIO1)
- new net MCUEncoderS: C11.1, R1.2, R19.2, U1.4 (GPIO2)
- no-connect marks 16 -> 25
Other:
- added sheet LED to RS485 (led-to-rs485.kicad_sch)
- added sheet LED to RS486 (led-to-rs485.kicad_sch)
- added sheet LED to RS487 (led-to-rs485.kicad_sch)
- added sheet LED to RS488 (led-to-rs485.kicad_sch)
- added sheet LED to RS489 (led-to-rs485.kicad_sch)
- added sheet LED to RS490 (led-to-rs485.kicad_sch)
- added sheet LED to RS491 (led-to-rs485.kicad_sch)
- added sheet LED to RS492 (led-to-rs485.kicad_sch)
- note added: "Front Panel Connector + Debounce"
- note added: "RS-485 Transmitters"
- note removed: "Connector to Front Panel"
- note removed: "LED 1 transmitter (RS485)"
- note removed: "LED 2 transmitter (RS485)"
- note removed: "LED 3 transmitter (RS485)"
- note removed: "LED 4 transmitter (RS485)"
- note removed: "LED 5 transmitter (RS485)"
- note removed: "LED 6 transmitter (RS485)"
- note removed: "LED 7 transmitter (RS485)"
- note removed: "LED 8 transmitter (RS485)"
- note removed: "current draw: ~500uA"
- moved on the sheet: C14, C15, C2, C3, H1, J1, J12, J13, J5, J8, JP1, JP2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

Commit message: 1st panel test, before cloning 8 receivers
Parts:
- removed C14: 220nF, Capacitor_SMD:C_0603_1608Metric, symbol Device:C_Small
- removed C15, C2: 100nF, Capacitor_SMD:C_0603_1608Metric, symbol Device:C_Small
- removed C3: 10uF, Capacitor_SMD:C_0402_1005Metric, symbol Device:C_Small
- removed H1: ~, Frangitron:frangitron_logo_16mm, symbol Frangitron:Frangitron_logo
- removed J12: ReceiverRS485, Frangitron:ScrewTerminal_01x03_5.08_Amphenol, symbol Connector:Screw_Terminal_01x03
- removed J8: ReceiverData, Frangitron:ScrewTerminal_01x02_5.08_Amphenol, symbol Connector:Screw_Terminal_01x02
- removed JP3: 1-2 12V, Jumper:SolderJumper-3_P2.0mm_Open_TrianglePad1.0x1.5mm_NumberLabels, symbol Jumper:SolderJumper_3_Open
- removed JP4: 12V, Jumper:SolderJumper-2_P1.3mm_Open_Pad1.0x1.5mm, symbol Jumper:SolderJumper_2_Open
- removed R10, R9: 20K, Resistor_SMD:R_0402_1005Metric, symbol Device:R_Small
- removed R6 (x2), R8: 10K, Resistor_SMD:R_0402_1005Metric, symbol Device:R_Small
- removed R7: 120, Resistor_SMD:R_0402_1005Metric, symbol Device:R_Small
- removed U13: LM7805, Package_TO_SOT_SMD:SOT-223, symbol Regulator_Linear:LM7805_TO220
- removed U4: MAX485E, Package_SO:SOIC-8_3.9x4.9mm_P1.27mm, symbol Interface_UART:MAX485E
- added H8, H9: MountingHole_Pad, MountingHole:MountingHole_3.2mm_M3_Pad, symbol Mechanical:MountingHole_Pad
Connections:
- net FP GND: now also H8.1, H9.1
Other:
- added sheet Receiver (Receiver.kicad_sch)
- note added: "current draw: ~200mA (sure ?)"
- note removed: "current draw: ~5.5mA"
- moved on the sheet: C11, C12, C13, C14, C15, C22, DS1, FM1, FM2, FM3, H1, H2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
