File: rp2040-led-board-schematics-v01.kicad_sch (KiCad schematic)
At the start: 53 parts, among them J27 MainBoard, J5 PWR_IN, J9 FrontPanel, Q1 AO3401A, SW1 PEC16, SW2 Button, U1 Pico, U2 LMR50410Y5FQDBVRQ1, U6 ENC28J60

Commit message: rename to v1 (to match silkscreen), improve readme and schematics layouts
Other:
- sheet LED to RS485 1 renamed Transmitter 1
- sheet LED to RS485 2 renamed Transmitter 2
- sheet LED to RS485 3 renamed Transmitter 3
- sheet LED to RS485 4 renamed Transmitter 4
- sheet LED to RS485 5 renamed Transmitter 5
- sheet LED to RS485 6 renamed Transmitter 6
- sheet LED to RS485 7 renamed Transmitter 7
- sheet LED to RS485 8 renamed Transmitter 8
- sheet Transmitter 1: file led-to-rs485.kicad_sch -> Transmitter.kicad_sch
- sheet Transmitter 2: file led-to-rs485.kicad_sch -> Transmitter.kicad_sch
- sheet Transmitter 3: file led-to-rs485.kicad_sch -> Transmitter.kicad_sch
- sheet Transmitter 4: file led-to-rs485.kicad_sch -> Transmitter.kicad_sch
- sheet Transmitter 5: file led-to-rs485.kicad_sch -> Transmitter.kicad_sch
- sheet Transmitter 6: file led-to-rs485.kicad_sch -> Transmitter.kicad_sch
- sheet Transmitter 7: file led-to-rs485.kicad_sch -> Transmitter.kicad_sch
- sheet Transmitter 8: file led-to-rs485.kicad_sch -> Transmitter.kicad_sch
- moved on the sheet: C11, C33, C34, C35, C36, C71, C72, C74, DS1, F1, FB2, FM1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
